File: schematics/car.kicad_pcb (KiCad board)
At the start: 2 copper layers, 30 parts, among them J1 Screw_Terminal_01x02, J2 Screw_Terminal_01x02, J3 Screw_Terminal_01x02, M1 Motor_Servo, Q1 2N3904, SW1 SW_SPDT, U1 L7805, U2 LM386, U3 LM386, U4 L293D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

Commit message: update layout
Parts:
- moved C4 10.2 mm to (119.4, 101.6)
- moved Q1 5.08 mm to (160.0, 114.3), turned to 270 degrees
Connections:
- Q1 pad 1: /SERVO -> Net-(M1-Pad1)
- Q1 pad 3: Net-(M1-Pad1) -> GND
- R8 pad 1: +3V3 -> /SERVO
- U1 pad 1: +BATT -> Net-(Q2-Pad2)
Routing:
- net GND: track 186.5 -> 209.1 mm
- net +3V3: track 34.6 -> 21.0 mm
- net +BATT: track 33.8 -> 21.5 mm
- net /SERVO: track 11.1 -> 16.1 mm

Commit message: voice streaming test
Connections:
- Q1 pad 1: Net-(M1-Pad1) -> /SERVO
- Q1 pad 3: GND -> Net-(M1-Pad1)
- R8 pad 1: /SERVO -> +3V3
- U1 pad 1: Net-(Q2-Pad2) -> +BATT
Routing:
- net +BATT: track 21.5 -> 35.5 mm
- net /SERVO: track 16.1 -> 22.3 mm
